Commit message: added green colour to robot.xacro

File: description/robot_core.xacro (robot description, xacro)
@@ -17,4 +17,7 @@
     <material name="red">
         <color rgba="1 0 0 1 " />
+    </material>
+    <material name="green">
+        <color rgba="0 1 0 1 " />
     </material>
 <!-- BASE LINK -->
